Commit message: ...

File: assets/biped2d.urdf (robot description, URDF)
Before this commit: robot balance, 10 links, 9 joints
Joints:
- joint l_ankle: limit lower=-1.6 upper=1. effort=10.0 velocity=1000.0 -> lower=-1. upper=0.5 effort=100.0 velocity=10.0
- joint l_knee: limit lower=-1.97. upper=0.1 effort=10.0 velocity=1000.0 -> lower=-1.57. upper=0.1 effort=300.0 velocity=15.0
- joint r_ankle: limit lower=-1.6 upper=1. effort=10.0 velocity=1000.0 -> lower=-1. upper=0.5 effort=100.0 velocity=10.0
- joint r_knee: limit lower=-1.97. upper=0.1 effort=10.0 velocity=1000.0 -> lower=-1.57. upper=0.1 effort=300.0 velocity=15.0
- joint torso_to_leftleg: limit lower=-1.77. upper=1.77 effort=1000.0 velocity=1000.0 -> lower=-1.57. upper=1.57 effort=500.0 velocity=15.0
- joint torso_to_rightleg: limit lower=-1.77. upper=1.77 effort=1000.0 velocity=1000.0 -> lower=-1.57. upper=1.57 effort=500.0 velocity=15.0
- joint torso_to_z: limit (none) -> lower=-0.4 upper=0.1 effort=500.0 velocity=10.0; type continuous -> revolute
- joint y_to_world: limit lower=1 upper=-1 effort=0.0 velocity=1000.0 -> lower=1 upper=-1 effort=0.0 velocity=20.0
- joint z_to_y: limit lower=1 upper=-1 effort=0.0 velocity=1000.0 -> lower=1 upper=-1 effort=0.0 velocity=20.0

Commit message: ...

File: assets/biped2d.urdf (robot description, URDF)
Before this commit: robot balance, 10 links, 9 joints
Joints:
- joint l_ankle: limit lower=-1. upper=0.5 effort=100.0 velocity=10.0 -> lower=-1.57 upper=0.5 effort=100.0 velocity=10.0
- joint l_knee: limit lower=-1.57. upper=0.1 effort=300.0 velocity=15.0 -> lower=-1.57. upper=0.1 effort=300.0 velocity=10.0
- joint r_ankle: limit lower=-1. upper=0.5 effort=100.0 velocity=10.0 -> lower=-1.57 upper=0.5 effort=100.0 velocity=10.0
- joint r_knee: limit lower=-1.57. upper=0.1 effort=300.0 velocity=15.0 -> lower=-1.57. upper=0.1 effort=300.0 velocity=10.0
- joint torso_to_leftleg: limit lower=-1.57. upper=1.57 effort=500.0 velocity=15.0 -> lower=-1.57. upper=1.57 effort=500.0 velocity=10.0
- joint torso_to_rightleg: limit lower=-1.57. upper=1.57 effort=500.0 velocity=15.0 -> lower=-1.57. upper=1.57 effort=500.0 velocity=10.0
- joint torso_to_z: limit lower=-0.4 upper=0.1 effort=500.0 velocity=10.0 -> lower=-0.4 upper=0.1 effort=500.0 velocity=5.0

Commit message: server running codes

File: assets/biped2d.urdf (robot description, URDF)
Before this commit: robot balance, 10 links, 9 joints
Joints:
- joint l_knee: limit lower=-1.57. upper=0.1 effort=300.0 velocity=15.0 -> lower=-1.57. upper=0.1 effort=300.0 velocity=10.0
- joint r_knee: limit lower=-1.57. upper=0.1 effort=300.0 velocity=15.0 -> lower=-1.57. upper=0.1 effort=300.0 velocity=10.0
- joint torso_to_leftleg: limit lower=-1.57. upper=1.57 effort=500.0 velocity=15.0 -> lower=-1.57. upper=1.57 effort=500.0 velocity=10.0
- joint torso_to_rightleg: limit lower=-1.57. upper=1.57 effort=500.0 velocity=15.0 -> lower=-1.57. upper=1.57 effort=500.0 velocity=10.0
- joint torso_to_z: limit lower=-0.4 upper=0.1 effort=500.0 velocity=10.0 -> lower=-0.4 upper=0.1 effort=500.0 velocity=5.0

Commit message: ordered and ready to run hyperparam tuning

File: assets/biped2d.urdf (robot description, URDF)
Before this commit: robot balance, 10 links, 9 joints
Joints:
- joint l_ankle: limit lower=-1. upper=0.5 effort=100.0 velocity=10.0 -> lower=-1.57 upper=0.5 effort=100.0 velocity=10.0
- joint r_ankle: limit lower=-1. upper=0.5 effort=100.0 velocity=10.0 -> lower=-1.57 upper=0.5 effort=100.0 velocity=10.0

Commit message: 21 july uptodate

File: assets/biped2d.urdf (robot description, URDF)
Before this commit: robot balance, 10 links, 9 joints
Joints:
- joint l_ankle: limit lower=-1.57 upper=0.5 effort=100.0 velocity=10.0 -> lower=-1.57 upper=0.5 effort=150.0 velocity=10.0
- joint l_knee: limit lower=-1.57. upper=0.1 effort=300.0 velocity=10.0 -> lower=-1.57 upper=0.1 effort=300.0 velocity=10.0
- joint r_ankle: limit lower=-1.57 upper=0.5 effort=100.0 velocity=10.0 -> lower=-1.57 upper=0.5 effort=150.0 velocity=10.0
- joint r_knee: limit lower=-1.57. upper=0.1 effort=300.0 velocity=10.0 -> lower=-1.57 upper=0.1 effort=300.0 velocity=10.0
- joint torso_to_leftleg: limit lower=-1.57. upper=1.57 effort=500.0 velocity=10.0 -> lower=-1.57 upper=1.57 effort=500.0 velocity=10.0

Commit message: improvements up to 28.08

File: assets/biped2d.urdf (robot description, URDF)
Before this commit: robot balance, 10 links, 9 joints
Joints:
- joint torso_to_z: limit lower=-0.4 upper=0.1 effort=500.0 velocity=5.0 -> lower=-1.01 upper=1.01 effort=500.0 velocity=5.0
